Commit message: Added velodyne 32channel lidar

File: urdf/flying_car.urdf.xacro (robot description, xacro)
@@ -933,3 +933,14 @@
       xyz="1 0 0" />
   </joint>
+  <xacro:include filename="$(find velodyne_description)/urdf/HDL-32E.urdf.xacro"/>
+  <xacro:HDL-32E
+    parent="base_link"
+    name="velodyne2"
+    topic="/velodyne_points2"
+    organize_cloud="false"
+    hz="10"
+    samples="220"
+    gpu="false">
+    <origin xyz="0.5 0 0.5" rpy="0 0 0" />
+  </xacro:HDL-32E>
 </robot>
