Commit message: Added prop joint controller

File: urdf/flying_car.gazebo.xacro (robot description, xacro)
@@ -19,4 +19,15 @@
     </transmission>
   </xacro:macro>
+  <xacro:macro name="SimpleTransmissionVelocity" params="joint n">
+    <transmission name="tran${n}">
+      <type>transmission_interface/SimpleTransmission</type>
+      <joint name="${joint}">
+        <hardwareInterface>hardware_interface/EffortJointInterface</hardwareInterface>
+      </joint>
+      <actuator name="${n}">
+        <mechanicalReduction>1</mechanicalReduction>
+      </actuator>
+    </transmission>
+  </xacro:macro>
   <xacro:SimpleTransmissionPosition n="1" joint="FL_steer_joint" />
   <xacro:SimpleTransmissionPosition n="2" joint="FR_steer_joint" />
@@ -25,3 +36,11 @@
   <xacro:SimpleTransmissionPosition n="5" joint="RL_arm_joint" />
   <xacro:SimpleTransmissionPosition n="6" joint="RR_arm_joint" />
+  <xacro:SimpleTransmissionPosition n="FL_prop" joint="FL_prop_joint" />
+  <xacro:SimpleTransmissionPosition n="FR_prop" joint="FR_prop_joint" />
+  <xacro:SimpleTransmissionPosition n="RL_prop" joint="RL_prop_joint" />
+  <xacro:SimpleTransmissionPosition n="RR_prop" joint="RR_prop_joint" />
+  <xacro:SimpleTransmissionVelocity n="FL_wheel" joint="FL_wheel_joint" />
+  <xacro:SimpleTransmissionVelocity n="FR_wheel" joint="FR_wheel_joint" />
+  <xacro:SimpleTransmissionVelocity n="RL_wheel" joint="RL_wheel_joint" />
+  <xacro:SimpleTransmissionVelocity n="RR_wheel" joint="RR_wheel_joint" />
 </robot>

File: urdf/flying_car.urdf.xacro (robot description, xacro)
@@ -144,6 +144,6 @@
   </link>
   <joint
-    name="FL_prop_link"
-    type="revolute">
+    name="FL_prop_joint"
+    type="continuous">
     <origin
       xyz="0.76505 0 0.254"
@@ -155,9 +155,4 @@
     <axis
       xyz="0 1 0" />
-    <limit
-      lower="0"
-      upper="0"
-      effort="0"
-      velocity="0" />
   </joint>
   <link

Commit message: Added flying_car.sdf file

File: urdf/flying_car.gazebo.xacro (robot description, xacro)
@@ -44,3 +44,14 @@
   <xacro:SimpleTransmissionVelocity n="RL_wheel" joint="RL_wheel_joint" />
   <xacro:SimpleTransmissionVelocity n="RR_wheel" joint="RR_wheel_joint" />
+  <!-- Velodyne LiDAR macro -->
+  <xacro:include filename="$(find velodyne_description)/urdf/HDL-32E.urdf.xacro"/>
+  <xacro:HDL-32E
+    parent="base_link"
+    name="velodyne2"
+    topic="/velodyne_points2"
+    hz="10"
+    samples="220"
+    gpu="false">
+    <origin xyz="0.5 0 0.5" rpy="0 0 0" />
+  </xacro:HDL-32E>
 </robot>

File: urdf/flying_car.urdf.xacro (robot description, xacro)
@@ -3,6 +3,8 @@
      Commit Version: 1.6.0-1-g15f4949  Build Version: 1.6.7594.29634
      For more information, please see http://wiki.ros.org/sw_urdf_exporter -->
-<robot name="flying_car_urdf" xmlns:xacro="http://ros.org/wiki/xacro">
+<!--robot name="flying_car_urdf" xmlns:xacro="http://ros.org/wiki/xacro"-->
+<robot name="iris" xmlns:xacro="http://ros.org/wiki/xacro">
   <xacro:include filename="$(find flying_car_urdf)/urdf/flying_car.gazebo.xacro"/>
+  <xacro:include filename="$(find flying_car_urdf)/urdf/flying_car.px4.xacro"/>
   <link
     name="base_link">
@@ -585,4 +587,10 @@
           filename="package://flying_car_urdf/meshes/FR_wheel_link.STL" />
       </geometry>
+      <friction>
+        <ode>
+          <mu>0.68</mu>
+          <mu2>0.8</mu2>
+        </ode>
+      </friction>
     </collision>
   </link>
@@ -696,4 +704,10 @@
           filename="package://flying_car_urdf/meshes/FL_wheel_link.STL" />
       </geometry>
+      <friction>
+        <ode>
+          <mu>0.68</mu>
+          <mu2>0.8</mu2>
+        </ode>
+      </friction>
     </collision>
   </link>
@@ -807,4 +821,10 @@
           filename="package://flying_car_urdf/meshes/RR_wheel_link.STL" />
       </geometry>
+      <friction>
+        <ode>
+          <mu>0.68</mu>
+          <mu2>0.8</mu2>
+        </ode>
+      </friction>
     </collision>
   </link>
@@ -918,4 +938,10 @@
           filename="package://flying_car_urdf/meshes/RL_wheel_link.STL" />
       </geometry>
+      <friction>
+        <ode>
+          <mu>0.68</mu>
+          <mu2>0.8</mu2>
+        </ode>
+      </friction>
     </collision>
   </link>
@@ -933,13 +959,3 @@
       xyz="1 0 0" />
   </joint>
-  <xacro:include filename="$(find velodyne_description)/urdf/HDL-32E.urdf.xacro"/>
-  <xacro:HDL-32E
-    parent="base_link"
-    name="velodyne2"
-    topic="/velodyne_points2"
-    hz="10"
-    samples="220"
-    gpu="false">
-    <origin xyz="0.5 0 0.5" rpy="0 0 0" />
-  </xacro:HDL-32E>
 </robot>
